File: pcb-board/kicad-project/NiAudio.kicad_sch (KiCad schematic)
At the start: 13 parts

Commit message: ready schematic
Parts:
- added 6M-49S-SR1: Crystal, symbol Device:Crystal
- added AZ1117CH-3.3: AZ1117CH-3.3TRG1, DIODES_AZ1117CH-3.3TRG1_0, symbol 3.3:AZ1117CH-3.3TRG1
- added C-100uF-Tantalum1, C-100uF-Tantalum2, C-100uF-Tantalum3, C-100uF-Tantalum4, C-10uF2, C-1uF3, C-22uF1, C-30pF1, C-30pF2, C-30pF3: C, symbol Device:C
- added D1, D2, D7, D8: D1213A-02SR, Package_TO_SOT_SMD:SOT-143, symbol D1213A-02SR:D1213A-02SR
- added D10, D11, D12, D3, D4, D5, D9: LED, symbol Device:LED
- added F-0.5A1, F-0.5A2, F-0.5A3, F-0.5A4: Fuse, symbol Device:Fuse
- added J1: pad-VB+, symbol Connector:Conn_01x01_Male
- added J10, J11, J12: pad, symbol Connector:Conn_01x01_Male
- added J13, J14, J2: pad-VB-, symbol Connector:Conn_01x01_Male
- added J3: pad-5VB, symbol Connector:Conn_01x01_Male
- added J4: pad-Gnd, symbol Connector:Conn_01x01_Male
- added J5, J6, J7, J8: USB-host, symbol Connector:USB_A
- added J9: USB_B_Micro_charger, symbol Connector:USB_B_Micro
- added JP1, JP10, JP11, JP12, JP13, JP14, JP15, JP16, JP17, JP18, JP19, JP2, JP20, JP21, JP22, JP23, JP24, JP25, JP26, JP27, JP28, JP29, JP3, JP4, JP5, JP6, JP7, JP8, JP9: SolderJumper_2_Open, symbol Jumper:SolderJumper_2_Open
- added Q3, Q4: AO3415-Pch, symbol ao3415:AO3415
- added R-1, R-1.5k1, R-10K1, R-10K2, R-15k1, R-1k1, R-2.7K1, R-3k1, R-3k2, R-3k3, R-3k4: R, symbol Device:R
- added R2, R3: R-500, symbol Device:R
- added SW1: RESET-Btn, symbol Switch:SW_Push
- added U3: TUSB2036, Package_QFP:LQFP-32_7x7mm_P0.8mm, symbol Interface_USB:TUSB2036
- Q1, Q2: renamed from Q?; value AO3418 -> AO3418-Nch
- R1: renamed from R-500; value R -> R-500
- gave numbers to parts that had none: 6
- renumbered C-10uF to C-10uF1, C-1uF to C-1uF1, C-1uF to C-1uF2, R-6.2k to R-6.2k1
Connections:
- net GND: now also AZ1117CH-3.3.1 (GND), C-100uF-Tantalum1.2, C-100uF-Tantalum2.2, C-100uF-Tantalum3.2, C-100uF-Tantalum4.2, C-10uF2.2, C-1uF3.1, C-22uF1.2, C-30pF1.2, C-30pF2.1, C-30pF3.1, D1.1 (GND/Vn), D2.1 (GND/Vn), D7.1 (GND/Vn), D8.1 (GND/Vn), J4.1 (Pin_1), J5.4 (GND), J5.5 (Shield), J6.4 (GND), J6.5 (Shield), J7.4 (GND), J7.5 (Shield), J8.4 (GND), J8.5 (Shield), J9.5 (GND), J9.6 (Shield), JP19.1 (A), JP2.2 (B), JP21.1 (A), JP25.2 (B), JP28.2 (B), R-1.2, R-10K1.2, R-10K2.2, R-3k1.2, R-3k2.2, R-3k3.2, R-3k4.2, SW1.2, U3.28 (GND), U3.7 (GND); no longer BT1.2 (-)
- net at C-1uF1.2, U2.3 (VBAT), U2.4 (VBAT): now also JP3.2 (B); no longer BT1.1 (+), R-330.1
- net at R-6.2k1.2, U2.8 (VSS), U2.9 (VSS): now also JP6.2 (B); no longer Q2.2, U1.1 (VM)
- net 5VPC: no longer names the net of C-10uF1.1, C-1uF2.1, D6.2 (A), U2.1 (VDD), U2.2 (VDD)
- net 5VPC: now also JP11.1 (A)
- new net: D9.1 (K), R-3k1.1
- new net: D9.2 (A), U3.22 (NPINT0)
- new net: 6M-49S-SR1.1, C-30pF2.2, R-1.5k1.2
- new net: 6M-49S-SR1.2, C-30pF1.1, U3.30 (XTAL1/CLK48)
- new net: Q3.1, R-10K2.1
- new net: R-2.7K1.1, U1.1 (VM)
- new net: AZ1117CH-3.3.2 (OUTPUT), C-22uF1.1, JP16.1 (A)
- new net: AZ1117CH-3.3.3 (INPUT), C-10uF2.1, JP12.2 (B)
- new net: C-100uF-Tantalum2.1, F-0.5A2.2, JP4.1 (A)
- new net: D5.1 (K), R-1.1
- new net: JP9.1 (A), Q3.2
- new net: JP7.2 (B), Q3.3
- new net: JP27.1 (A), U3.14 (~{OVRCUR2})
- new net: J14.1 (Pin_1), JP27.2 (B)
- new net: D3.1 (K), R2.1
- new net: F-0.5A2.1, J6.1 (VBUS)
- new net: C-100uF-Tantalum4.1, F-0.5A4.2, JP15.1 (A)
- new net: F-0.5A1.1, J5.1 (VBUS)
- new net: C-100uF-Tantalum1.1, F-0.5A1.2, JP5.1 (A)
- new net: F-0.5A4.1, J8.1 (VBUS)
- new net: JP22.1 (A), U3.25 (VCC), U3.3 (VCC)
- new net: R-1k1.1, SW1.1
- new net: BT1.2 (-), JP2.1 (A)
- new net: BT1.1 (+), JP1.1 (A)
- new net: D10.1 (K), R-3k2.1
- new net: D10.2 (A), U3.23 (NPINT1)
- new net: C-1uF3.2, JP29.1 (A), R-15k1.1, R-1k1.2
- new net: J9.1 (VBUS), JP14.1 (A)
- new net: J11.1 (Pin_1), J9.2 (D-)
- new net: J10.1 (Pin_1), J9.3 (D+)
- new net: J12.1 (Pin_1), J9.4 (ID)
- new net: D4.1 (K), R3.1
- new net: JP18.2 (B), U3.21 (~{OCPROT}/~{PWRSW})
- new net: JP26.1 (A), U3.10 (~{OVRCUR1})
- new net: JP24.1 (A), U3.13 (~{PWRON2})
- new net: JP25.1 (A), U3.17 (~{PWRON3})
- new net: JP28.1 (A), U3.18 (~{OVRCUR3})
- new net: JP19.2 (B), U3.24 (~{NP3})
- new net: JP20.2 (B), U3.26 (~{EXTMEM})
- new net: D11.2 (A), U3.27 (DP0PUR)
- new net: R-1.5k1.1, U3.29 (XTAL2)
- new net: JP21.2 (B), U3.31 (MODE)
- new net: D12.2 (A), U3.32 (SUSPND)
- new net: JP17.2 (B), U3.8 (~{BUSPWR})
- new net: JP23.1 (A), U3.9 (~{PWRON1})
- new net: D11.1 (K), R-3k3.1
- new net: C-100uF-Tantalum3.1, F-0.5A3.2, JP13.1 (A)
- new net: J13.1 (Pin_1), JP24.2 (B)
- new net: JP10.1 (A), Q4.2
- new net: JP8.1 (A), Q4.3
- new net: F-0.5A3.1, J7.1 (VBUS)
- new net: D12.1 (K), R-3k4.1
- new net 3.3V: C-30pF3.2, JP16.2 (B), JP17.1 (A), JP18.1 (A), JP20.1 (A), JP22.2 (B), JP23.2 (B), JP26.2 (B), R-15k1.2
- new net 5VB: D4.2 (A), J3.1 (Pin_1), JP8.2 (B), R3.2
- new net 5VC: D3.2 (A), JP11.2 (B), JP14.2 (B), JP7.1 (A), Q4.1, R-10K1.1, R2.2
- new net 5VM: D1.4 (VCC/Vn), D2.4 (VCC/Vn), D5.2 (A), D7.4 (VCC/Vn), D8.4 (VCC/Vn), JP10.2 (B), JP12.1 (A), JP13.2 (B), JP15.2 (B), JP4.2 (B), JP5.2 (B), JP9.2 (B)
- new net RST: JP29.2 (B), U3.4 (~{RESET})
- new net USB-G1-minus: D1.2 (CH1), J5.2 (D-), U3.11 (DM1)
- new net USB-G1-plus: D1.3 (CH2), J5.3 (D+), U3.12 (DP1)
- new net USB-G2-minus: D7.2 (CH1), J7.2 (D-), U3.15 (DM2)
- new net USB-G2-plus: D7.3 (CH2), J7.3 (D+), U3.16 (DP2)
- new net USB-G3-minus: D8.2 (CH1), J8.2 (D-), U3.19 (DM3)
- new net USB-G3-plus: D8.3 (CH2), J8.3 (D+), U3.20 (DP3)
- new net USB-H-minus: D2.2 (CH1), J6.2 (D-), U3.2 (DM0)
- new net USB-H-plus: D2.3 (CH2), J6.3 (D+), U3.1 (DP0)
- new net VB+: J1.1 (Pin_1), JP1.2 (B), JP3.1 (A), R-330.1
- new net VB-: J2.1 (Pin_1), JP6.1 (A), Q2.2, R-2.7K1.2
Other:
- note added: "3.3V made"
- note added: "5V from cable"
- note added: "Battery charging"
- note added: "Battery protection"
- note added: "Leave untouched"
- note added: "Power source switching"
- note added: "Pull high"
- note added: "Reset circuit"
- note added: "USB hub"
- note added: "any step up converter board"

Commit message: footprints annotations
Parts:
- added C-100nF-Ceramic2: C, Capacitor_THT:C_Disc_D5.0mm_W2.5mm_P2.50mm, symbol Device:C
- added C-1uF2: C, Capacitor_THT:CP_Radial_D6.3mm_P2.50mm, symbol Device:C
- added D13: LED, LED_THT:LED_D3.0mm_Clear, symbol Device:LED
- added J15, J16: pad, TestPoint:TestPoint_Pad_2.0x2.0mm, symbol Connector:Conn_01x01_Male
- added R-3k2: R, Resistor_THT:R_Axial_DIN0414_L11.9mm_D4.5mm_P15.24mm_Horizontal, symbol Device:R
- 6M-49S-SR1: footprint (none) -> Crystal:Crystal_HC18-U_Vertical
- AZ1117CH-3.3: footprint DIODES_AZ1117CH-3.3TRG1_0 -> 3.3:DIODES_AZ1117CH-3.3TRG1_0
- BT1: footprint (none) -> Connector_JST:JST_PH_S2B-PH-K_1x02_P2.00mm_Horizontal
- C-100nF-Ceramic1: renamed from C-1uF2; footprint (none) -> Capacitor_THT:C_Disc_D5.0mm_W2.5mm_P2.50mm
- C-100nF1, C-30pF3: footprint (none) -> Capacitor_THT:C_Disc_D5.0mm_W2.5mm_P2.50mm
- C-100uF-Tantalum1, C-100uF-Tantalum2, C-100uF-Tantalum3, C-100uF-Tantalum4: footprint (none) -> Capacitor_Tantalum_SMD:CP_EIA-6032-28_Kemet-C_Pad2.25x2.35mm_HandSolder
- C-10uF1, C-10uF2, C-1uF1, C-1uF3, C-22uF1: footprint (none) -> Capacitor_THT:CP_Radial_D6.3mm_P2.50mm
- C-30pF-Ceramic1: renamed from C-30pF1; footprint (none) -> Capacitor_THT:C_Disc_D5.0mm_W2.5mm_P2.50mm
- C-30pF-Ceramic2: renamed from C-30pF2; footprint (none) -> Capacitor_THT:C_Disc_D5.0mm_W2.5mm_P2.50mm
- D10, D11, D12, D3, D4, D5, D6, D9: footprint (none) -> LED_THT:LED_D3.0mm_Clear
- F-0.5A1, F-0.5A2, F-0.5A3, F-0.5A4: footprint (none) -> Fuse:Fuse_0603_1608Metric_Pad1.05x0.95mm_HandSolder
- J1, J2, J3, J4: footprint (none) -> TestPoint:TestPoint_THTPad_4.0x4.0mm_Drill2.0mm
- J10, J11, J12, J13, J14: footprint (none) -> TestPoint:TestPoint_Pad_2.0x2.0mm
- J5, J6, J7, J8: footprint (none) -> Connector_USB:USB_A_Stewart_SS-52100-001_Horizontal
- J9: footprint (none) -> Connector_USB:USB_Micro-B_Amphenol_10118194_Horizontal
- JP1, JP10, JP11, JP12, JP13, JP14, JP15, JP16, JP17, JP18, JP19, JP2, JP20, JP21, JP22, JP23, JP24, JP25, JP26, JP27, JP28, JP29, JP3, JP4, JP5, JP6, JP7, JP8, JP9: footprint (none) -> Jumper:SolderJumper-2_P1.3mm_Open_Pad1.0x1.5mm
- Q1, Q2, Q3, Q4: footprint (none) -> mosfet:SOT-23
- R-1.5k1, R-10K1, R-10K2, R-15k1, R-1k1, R-2.7K1, R-330, R-3k4, R-6.2k1: footprint (none) -> Resistor_THT:R_Axial_DIN0414_L11.9mm_D4.5mm_P15.24mm_Horizontal
- R-3k1: renamed from R-1; footprint (none) -> Resistor_THT:R_Axial_DIN0414_L11.9mm_D4.5mm_P15.24mm_Horizontal
- R-3k3: renamed from R-3k1; footprint (none) -> Resistor_THT:R_Axial_DIN0414_L11.9mm_D4.5mm_P15.24mm_Horizontal
- R-3k5: renamed from R-3k2; footprint (none) -> Resistor_THT:R_Axial_DIN0414_L11.9mm_D4.5mm_P15.24mm_Horizontal
- R-3k6: renamed from R-3k3; footprint (none) -> Resistor_THT:R_Axial_DIN0414_L11.9mm_D4.5mm_P15.24mm_Horizontal
- R1, R2, R3: value R-500 -> R-3k; footprint (none) -> Resistor_THT:R_Axial_DIN0414_L11.9mm_D4.5mm_P15.24mm_Horizontal
- SW1: footprint (none) -> Button_Switch_THT:SW_PUSH_6mm
- U2: footprint Microchip-MCP73113-06SI_MF-* -> eec:Microchip-MCP73113-06SI_MF-Manufacturer_Recommended
Connections:
- net GND: now also C-100nF-Ceramic2.2, C-1uF2.1, R-3k2.2
- net at AZ1117CH-3.3.2 (OUTPUT), C-22uF1.1, JP16.1 (A): now also D13.2 (A)
- net at JP22.1 (A), U3.25 (VCC), U3.3 (VCC): now also C-100nF-Ceramic2.1, C-1uF2.2
- net at BT1.2 (-), JP2.1 (A): now also J16.1 (Pin_1)
- net at BT1.1 (+), JP1.1 (A): now also J15.1 (Pin_1)
- new net: D13.1 (K), R-3k2.1

Commit message: almost ready pcb
Parts:
- removed J6: USB-host, Connector_USB:USB_A_Stewart_SS-52100-001_Horizontal, symbol Connector:USB_A
- removed JP24, JP27: SolderJumper_2_Open, Jumper:SolderJumper-2_P1.3mm_Open_Pad1.0x1.5mm, symbol Jumper:SolderJumper_2_Open
- added J6: USB_B_Host, Connector_USB:USB_Micro-B_Amphenol_10118194_Horizontal, symbol Connector:USB_B_Micro
- C-30pF-Ceramic1, C-30pF-Ceramic2: footprint Capacitor_THT:C_Disc_D5.0mm_W2.5mm_P2.50mm -> Capacitor_SMD:C_1812_4532Metric_Pad1.57x3.40mm_HandSolder
- J1, J2, J3, J4: footprint TestPoint:TestPoint_THTPad_4.0x4.0mm_Drill2.0mm -> TestPoint:TestPoint_THTPad_1.5x1.5mm_Drill0.7mm
- R-1.5k1, R-10K1, R-10K2, R-15k1, R-1k1, R-2.7K1, R-330, R-3k1, R-3k2, R-3k3, R-3k4, R-3k5, R-3k6, R-6.2k1, R1, R2, R3: footprint Resistor_THT:R_Axial_DIN0414_L11.9mm_D4.5mm_P15.24mm_Horizontal -> Resistor_SMD:R_1812_4532Metric_Pad1.30x3.40mm_HandSolder
Connections:
- net VB- is gone; now on net GND: J2.1 (Pin_1), JP6.1 (A), Q2.2, R-2.7K1.2
- net 5VB: no longer R3.2
- net 5VC: no longer R2.2
- net GND: now also R2.2, R3.2, J6.5 (GND), J6.6 (Shield); no longer C-100nF1.1, JP2.2 (B), Q1.2, U1.3 (VSS)
- net USB-H-minus: now also J6.2 (D-)
- net USB-H-plus: now also J6.3 (D+)
- net at U3.14 (~{OVRCUR2}): now also J14.1 (Pin_1)
- net at F-0.5A2.1: now also J6.1 (VBUS)
- net at U3.13 (~{PWRON2}): now also J13.1 (Pin_1)
- new net: C-100nF1.1, JP2.2 (B), Q1.2, U1.3 (VSS)
