File: pcb-board/kicad-project/NiAudio.kicad_pcb (KiCad board)
At the start: 2 copper layers, 106 parts, among them J1 pad-VB+, J10 pad, J11 pad, J12 pad, J13 pad-VB-, J14 pad-VB-, J15 pad, J16 pad, J2 pad-VB-, J3 pad-5VB, J4 pad-Gnd, J5 USB-host, J6 USB-host, J7 USB-host, J8 USB-host, J9 USB_B_Micro_charger, Q1 AO3418-Nch, Q2 AO3418-Nch, Q3 AO3415-Pch, Q4 AO3415-Pch, SW1 RESET-Btn, U1 AP9101CK, U2 MCP73113-06SI_MF, U3 TUSB2036

Commit message: almost ready pcb
Parts:
- removed JP24, JP27: SolderJumper_2_Open, Jumper:SolderJumper-2_P1.3mm_Open_Pad1.0x1.5mm
- C-30pF-Ceramic1, C-30pF-Ceramic2: footprint Capacitor_THT:C_Disc_D5.0mm_W2.5mm_P2.50mm -> Capacitor_SMD:C_1812_4532Metric_Pad1.57x3.40mm_HandSolder
- J1, J2, J3, J4: footprint TestPoint:TestPoint_THTPad_4.0x4.0mm_Drill2.0mm -> TestPoint:TestPoint_THTPad_1.5x1.5mm_Drill0.7mm
- J6: value USB-host -> USB_B_Host; footprint Connector_USB:USB_A_Stewart_SS-52100-001_Horizontal -> Connector_USB:USB_Micro-B_Amphenol_10118194_Horizontal
- R-1.5k1, R-10K1, R-10K2, R-15k1, R-1k1, R-2.7K1, R-330, R-3k1, R-3k2, R-3k3, R-3k4, R-3k5, R-3k6, R-6.2k1, R1, R2, R3: footprint Resistor_THT:R_Axial_DIN0414_L11.9mm_D4.5mm_P15.24mm_Horizontal -> Resistor_SMD:R_1812_4532Metric_Pad1.30x3.40mm_HandSolder
- moved R-3k5 170.3 mm to (195.8, 31.6)
- moved R-3k6 158.9 mm to (185.4, 30.4), turned to 90 degrees
- moved R-3k3 148.5 mm to (195.8, 36.2)
- moved D11 142.0 mm to (185.4, 34.7), turned to -90 degrees
- moved D10 117.6 mm to (191.5, 31.6), turned to 180 degrees
- moved 6M-49S-SR1 116.4 mm to (132.6, 54.8), turned to 180 degrees
- moved J5 115.2 mm to (154.3, 80.9), turned to 90 degrees
- moved JP20 112.5 mm to (182.0, 57.4)
- moved C-100uF-Tantalum3 111.1 mm to (150.1, 58.2), turned to -90 degrees
- moved D9 106.5 mm to (188.9, 36.2)
- moved C-100uF-Tantalum1 103.5 mm to (148.5, 84.5)
- moved JP2 93.0 mm to (103.0, 35.8), turned to -90 degrees
- moved D8 93.0 mm to (144.2, 46.7), turned to 180 degrees
- moved R-15k1 87.2 mm to (124.2, 86.8), turned to -90 degrees
- moved C-1uF2 86.6 mm to (121.2, 58.1), turned to -90 degrees
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Connections:
- net /USB-G1-minus renamed /G1-
- net /USB-G1-plus renamed /G1+
- net /USB-G2-minus renamed /G2-
- net /USB-G2-plus renamed /G2+
- net /USB-G3-minus renamed /G3-
- net /USB-G3-plus renamed /G3+
- net /USB-H-minus renamed /H-
- net /USB-H-plus renamed /H+
- C-100nF1 pad 1: GND -> Net-(C-100nF1-Pad1)
- J2 pad 1: /VB- -> GND
- J6 pad 4: GND -> unconnected-(J6-Pad4)
- JP2 pad 2: GND -> Net-(C-100nF1-Pad1)
- JP6 pad 1: /VB- -> GND
- Q1 pad 2: GND -> Net-(C-100nF1-Pad1)
- Q2 pad 2: /VB- -> GND
- R-2.7K1 pad 2: /VB- -> GND
- R2 pad 2: /5VC -> GND
- R3 pad 2: /5VB -> GND
- U1 pad 3: GND -> Net-(C-100nF1-Pad1)
- U3 pad 13: Net-(JP24-Pad1) -> Net-(J13-Pad1)
- U3 pad 14: Net-(JP27-Pad1) -> Net-(J14-Pad1)
Routing:
- net /VB+: track 0.00 -> 63.8 mm, vias 0 -> 1
- net /H+: track 0.00 -> 54.2 mm
- net /H-: track 0.00 -> 54.2 mm
- net /5VB: track 0.00 -> 46.6 mm
- net Net-(JP6-Pad2): track 0.00 -> 41.7 mm
- net /5VC: track 0.00 -> 36.5 mm, vias 0 -> 2
- net /G2+: track 0.00 -> 33.1 mm
- net /G2-: track 0.00 -> 33.0 mm
- net /G1-: track 0.00 -> 30.6 mm
- net /G1+: track 0.00 -> 30.6 mm
- net /3.3V: track 0.00 -> 30.3 mm
- net /5VM: track 0.00 -> 29.3 mm, vias 0 -> 1
- net Net-(C-100nF1-Pad1): track 0.00 -> 25.1 mm, vias 0 -> 2
- net /G3+: track 0.00 -> 25.0 mm
- net /G3-: track 0.00 -> 24.9 mm
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- added copper zone on B.Cu, net GND
- added copper zone on F.Cu, net GND
Other:
- board outline added: 99 x 75.7 mm
- board text added: "+"
- board text added: "-"
- board text added: "3.3V Converter"
- board text added: "Baterry Protector"
- board text added: "Battery charger"
- board text added: "Power source switching"

Commit message: pcb finish
Parts:
- J2: value pad-VB- -> VB-
- J3: value pad-5VB -> 5VB
- J4: value pad-Gnd -> Gnd
- moved D11 53.7 mm to (132.1, 41.2)
- moved R-3k 53.7 mm to (132.1, 36.9)
- moved D10 43.8 mm to (159.0, 61.0)
- moved R-3k 43.8 mm to (163.3, 61.0)
- moved R-3k 43.8 mm to (163.3, 65.6)
- moved D9 42.0 mm to (159.0, 65.6), turned to 180 degrees
- moved J14 38.1 mm to (140.2, 72.8)
- moved JP19 37.7 mm to (144.6, 65.1), turned to 90 degrees
- moved JP18 37.6 mm to (144.8, 68.1)
- moved JP28 37.5 mm to (144.8, 70.6)
- moved JP25 37.5 mm to (144.8, 73.1)
- moved JP20 35.5 mm to (146.9, 62.7), turned to 90 degrees
- moved SW1 4.52 mm to (124.3, 95.0), turned to -90 degrees
- moved JP23 2.70 mm to (130.2, 73.3)
- moved JP26 2.40 mm to (132.7, 73.3)
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- renumbered 6M-49S-SR1 to 6M-49S-SR, C-100nF-Ceramic1 to C-100nF-Ceramic, C-100nF-Ceramic2 to C-100nF-Ceramic, C-100uF-Tantalum1 to C-100uF-Tantalum, C-100uF-Tantalum3 to C-100uF-Tantalum, C-100uF-Tantalum4 to C-100uF-Tantalum, C-100uF-Tantalum2 to C-100uF-Tantalum, C-10uF2 to C-10uF, C-10uF1 to C-10uF, C-1uF1 to C-1uF, C-1uF2 to C-1uF, C-22uF1 to C-22uF, C-30pF3 to C-30pF, C-30pF-Ceramic1 to C-30pF-Ceramic, C-30pF-Ceramic2 to C-30pF-Ceramic, F-0.5A4 to F-0.5A, F-0.5A3 to F-0.5A, F-0.5A1 to F-0.5A, F-0.5A2 to F-0.5A, R-1.5k1 to R-1.5k, R-10K2 to R-10K, R-10K1 to R-10K, R-15k1 to R-15k, R-1k1 to R-1k, R-2.7K1 to R-2.7K, R-3k3 to R-3k, R-3k2 to R-3k, R-3k6 to R-3k, R-3k5 to R-3k, R-3k4 to R-3k, R-6.2k1 to R-6.2k
Routing:
- net /5VM: track 29.3 -> 183.6 mm, vias 1 -> 10
- net /3.3V: track 30.3 -> 83.9 mm, vias 0 -> 4
- net GND: track 23.9 -> 75.9 mm, vias 4 -> 12
- net Net-(C-100uF-Tantalum4-Pad1): track 0.00 -> 26.6 mm
- net /RST: track 0.00 -> 25.5 mm, vias 0 -> 2
- net Net-(D9-Pad2): track 0.00 -> 24.2 mm, vias 0 -> 1
- net Net-(D11-Pad2): track 0.00 -> 23.3 mm, vias 0 -> 1
- net Net-(C-100nF-Ceramic2-Pad1): track 5.83 -> 26.3 mm, vias 0 -> 2
- net Net-(D10-Pad2): track 0.00 -> 20.0 mm, vias 0 -> 1
- net Net-(JP20-Pad2): track 0.00 -> 18.6 mm, vias 0 -> 2
- net Net-(JP19-Pad2): track 0.00 -> 17.2 mm, vias 0 -> 2
- net Net-(JP18-Pad2): track 0.00 -> 15.4 mm, vias 0 -> 2
- net Net-(J14-Pad1): track 0.00 -> 12.0 mm, vias 0 -> 2
- net Net-(D12-Pad2): track 0.00 -> 11.2 mm
- net Net-(JP25-Pad1): track 0.00 -> 11.2 mm, vias 0 -> 2
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Other:
- board text added: "VB+"

Commit message: minor things
Parts:
- F-0.5A (x4): footprint Fuse:Fuse_0603_1608Metric_Pad1.05x0.95mm_HandSolder -> Fuse:Fuse_1210_3225Metric_Pad1.42x2.65mm_HandSolder
- moved C-100uF-Tantalum 2.97 mm to (150.4, 61.1)
- moved F-0.5A 1.37 mm to (151.3, 54.6), turned to -90 degrees
- moved JP5 0.88 mm to (146.7, 80.9)
- moved F-0.5A 0.87 mm to (140.4, 97.8)
- moved JP13 0.71 mm to (153.8, 58.3)
- moved F-0.5A 0.47 mm to (147.5, 47.1)
Routing:
- net Net-(F-0.5A2-Pad1): track 4.24 -> 3.31 mm
- net Net-(C-100uF-Tantalum1-Pad1): track 6.47 -> 7.26 mm
- net Net-(F-0.5A1-Pad1): track 2.50 -> 1.89 mm
- net Net-(C-100uF-Tantalum4-Pad1): track 26.6 -> 27.2 mm
- net Net-(C-100uF-Tantalum3-Pad1): track 6.24 -> 6.79 mm
- net Net-(JP6-Pad2): track 41.7 -> 42.2 mm
- net Net-(F-0.5A3-Pad1): track 2.67 -> 3.18 mm
- net /5VM: track 183.6 -> 183.1 mm, vias 10 -> 9
